File: Monotech-HD-Floppy-Serial.sch (KiCad schematic (older format))
At the start: 42 parts, among them P1 Floppy, P2 Serial Port, SW1 Serial Port Config, SW2 Boot ROM Address, SW3 Enable ROM, SW4 ROM Write-Protect, SW5 28C64B Mode, U1 82077AA/PC8477, U2 16(C)x50, U3 GD75232/75(C)185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

Commit message: Add files via upload
Parts:
- SW1: footprint Buttons_Switches_THT:SW_DIP_x8_W7.62mm_Slide_LowProfile -> Buttons_Switches_THT:SW_DIP_x8_W7.62mm_Slide
- SW2: footprint Buttons_Switches_THT:SW_DIP_x4_W7.62mm_Slide_LowProfile -> Buttons_Switches_THT:SW_DIP_x4_W7.62mm_Slide
Changed lines of the file:
@@
 F 0 "SW1" H 7300 2967 50  0000 C CNN
 F 1 "Serial Port Config" H 7300 2876 50  0000 C CNN
-F 2 "Buttons_Switches_THT:SW_DIP_x8_W7.62mm_Slide_LowProfile" H 7300 2300 50  0001 C CNN
+F 2 "Buttons_Switches_THT:SW_DIP_x8_W7.62mm_Slide" H 7300 2300 50  0001 C CNN
 F 3 "" H 7300 2300 50  0001 C CNN
 	1    7300 2300
@@
 F 0 "SW2" H 1850 5150 50  0000 C CNN
 F 1 "Boot ROM Address" H 1850 5250 50  0000 C CNN
-F 2 "Buttons_Switches_THT:SW_DIP_x4_W7.62mm_Slide_LowProfile" H 1850 5500 50  0001 C CNN
+F 2 "Buttons_Switches_THT:SW_DIP_x4_W7.62mm_Slide" H 1850 5500 50  0001 C CNN
 F 3 "" H 1850 5500 50  0001 C CNN
 	1    1850 5500
