File: Monotech-HD-Floppy-Serial.kicad_pcb (KiCad board)
At the start: 2 copper layers, 105.4 x 83.8 mm, 43 parts, among them P1 Floppy, P2 Serial Port, SW1 Serial Port Config, SW2 Boot ROM Address, SW3 Enable ROM, SW4 ROM Write-Protect, SW5 28C64B Mode, U1 82077AA/PC8477, U2 16(C)x50, U3 GD75232/75(C)185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

Commit message: Add files via upload
Parts:
- SW1: footprint Buttons_Switches_THT:SW_DIP_x8_W7.62mm_Slide_LowProfile -> Buttons_Switches_THT:SW_DIP_x8_W7.62mm_Slide
- SW2: footprint Buttons_Switches_THT:SW_DIP_x4_W7.62mm_Slide_LowProfile -> Buttons_Switches_THT:SW_DIP_x4_W7.62mm_Slide
Other:
- board text added: "1 2 3 4"
- board text added: "1 2 3 4 5 6 7 8"
- board text added: "Boot ROM Address"
- board text added: "Serial Port Config"

Commit message: Add files via upload
Parts:
- BUS1: footprint Conn_Bus_ISA8 -> Custom:Conn_Bus_ISA8
- moved G*** 9.13 mm to (200.0, 147.7)
Other:
- board text added: "Monotech DeluxeFloppy Bootable ISA HD-Floppy + Serial Controller Card"
- board text added: "ROM > Write-Protect"
- board text added: "ROM Enable>"
- board text added: "Rev 1.1"
- board text removed: "< ROM Write-Protect"
- board text removed: "<ROM Enable"
- board text removed: "ISA HD-Floppy+Serial Controller Card Rev1.1 ----- Monotech PCs"
